Commit message: not req

File: mars_gazebo/unitree_g1/g1_gazebo.urdf (robot description, URDF)
Before this commit: robot g1_29dof_mode_15_brainco_hand, 73 links, 72 joints
Links:
- added link height_scanner_link
Joints:
- added joint height_scanner_joint: type fixed, parent pelvis, child height_scanner_link, origin xyz=0 0 -0.05 rpy=0 0 0

Commit message: Final corrected env with height scanner

File: mars_gazebo/unitree_g1/g1_gazebo.urdf (robot description, URDF)
Before this commit: robot g1_29dof_mode_15_brainco_hand, 74 links, 73 joints
Joints:
- joint height_scanner_joint: origin xyz=0 0 -0.05 rpy=0 0 0 -> xyz=0 0 0 rpy=3.14159 0 0
